Commit message: updated

File: description/robot_core.xacro (robot description, xacro)
@@ -109,3 +109,19 @@
         </xacro:inertial_sphere>
     </link>
+    <!-- ROS 2 Control -->
+<ros2_control name="ros2_control" type="system">
+  <hardware>
+    <plugin>gazebo_ros2_control/GazeboSystem</plugin>
+  </hardware>
+  <joint name="left_wheel_joint">
+    <command_interface name="velocity"/>
+    <state_interface name="position"/>
+    <state_interface name="velocity"/>
+  </joint>
+  <joint name="right_wheel_joint">
+    <command_interface name="velocity"/>
+    <state_interface name="position"/>
+    <state_interface name="velocity"/>
+  </joint>
+</ros2_control>
 </robot>
